File: Electronics/LightSchematic.sch (EAGLE design)
At the start: 7 parts, among them IC1 7805T, IC2 ATMEGA328-20P

Commit message: Add v0.2.1 for milestone 4 review
Connections:
- net DIN: now also IC2.(PCI18/INT0)PD2; no longer IC2.(PCI16/RXD)PD0
Changed lines of the file:
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@@
 <junction x="-83.82" y="139.7"/>
 <wire x1="-83.82" y1="139.7" x2="-40.64" y2="139.7" width="0.1524" layer="91"/>
-<pinref part="IC2" gate="G$1" pin="(PCI16/RXD)PD0"/>
-<wire x1="-40.64" y1="139.7" x2="-40.64" y2="86.36" width="0.1524" layer="91"/>
-<wire x1="-40.64" y1="86.36" x2="-48.26" y2="86.36" width="0.1524" layer="91"/>
+<wire x1="-40.64" y1="139.7" x2="-40.64" y2="83.82" width="0.1524" layer="91"/>
 <label x="-78.74" y="139.7" size="1.778" layer="95" rot="R90" xref="yes"/>
+<pinref part="IC2" gate="G$1" pin="(PCI18/INT0)PD2"/>
+<wire x1="-48.26" y1="81.28" x2="-43.18" y2="81.28" width="0.1524" layer="91"/>
+<wire x1="-43.18" y1="81.28" x2="-40.64" y2="83.82" width="0.1524" layer="91"/>
 </segment>
 </net>

Commit message: Added 16 MHz crystal oscillator and 2 22 pF capacitors
Parts:
- added C1, C2: 22pF, SparkFun-Capacitors:22PF-0603-50V-5%
- added Y1: 16MHz, SparkFun-Clocks:CRYSTAL-16MHZPTH-HC49US
- R1: value 100K -> 4.7k
- R2: value 100K -> 150
Connections:
- new net N$1: C1.1, IC2.PB6(XTAL1/TOSC1/PCI6), Y1.1
- new net N$2: C2.1, IC2.PB7(XTAL2/TOSC2/PCI7), Y1.2
- net GND: now also C1.2, C2.2
Other:
- moved on the sheet: G1, IC1
Changed lines of the file:
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@@
 </classes>
 <parts>
-<part name="R1" library="SparkFun-Resistors" library_urn="urn:adsk.eagle:library:532" deviceset="100KOHM" device="-0402-1/16W-1%" package3d_urn="urn:adsk.eagle:package:39657/1" value="100K"/>
+<part name="R1" library="SparkFun-Resistors" library_urn="urn:adsk.eagle:library:532" deviceset="100KOHM" device="-0402-1/16W-1%" package3d_urn="urn:adsk.eagle:package:39657/1" value="4.7k"/>
 <part name="G1" library="battery" library_urn="urn:adsk.eagle:library:109" deviceset="AB9V" device="" package3d_urn="urn:adsk.eagle:package:4600/1"/>
 <part name="IC1" library="linear" library_urn="urn:adsk.eagle:library:262" deviceset="78*" device="T" package3d_urn="urn:adsk.eagle:package:16414/1" technology="05"/>
-<part name="R2" library="SparkFun-Resistors" library_urn="urn:adsk.eagle:library:532" deviceset="100KOHM" device="-0402-1/16W-1%" package3d_urn="urn:adsk.eagle:package:39657/1" value="100K"/>
+<part name="R2" library="SparkFun-Resistors" library_urn="urn:adsk.eagle:library:532" deviceset="100KOHM" device="-0402-1/16W-1%" package3d_urn="urn:adsk.eagle:package:39657/1" value="150"/>
 <part name="D1" library="SparkFun-LED" library_urn="urn:adsk.eagle:library:529" deviceset="LED" device="1206" package3d_urn="urn:adsk.eagle:package:39352/1"/>
 <part name="S1" library="adafruit" library_urn="urn:adsk.eagle:library:420" deviceset="SPST" device="" package3d_urn="urn:adsk.eagle:package:6240821/1"/>
 <part name="IC2" library="atmega328" deviceset="ATMEGA328*P" device="" technology="-20"/>
+<part name="Y1" library="SparkFun-Clocks" library_urn="urn:adsk.eagle:library:511" deviceset="CRYSTAL-16MHZ" device="PTH-HC49US" package3d_urn="urn:adsk.eagle:package:37515/1" value="16MHz"/>
+<part name="C1" library="SparkFun-Capacitors" library_urn="urn:adsk.eagle:library:510" deviceset="22PF" device="-0603-50V-5%" package3d_urn="urn:adsk.eagle:package:37414/1" value="22pF"/>
+<part name="C2" library="SparkFun-Capacitors" library_urn="urn:adsk.eagle:library:510" deviceset="22PF" device="-0603-50V-5%" package3d_urn="urn:adsk.eagle:package:37414/1" value="22pF"/>
 </parts>
 <sheets>
@@
 <attribute name="VALUE" x="-82.296" y="134.62" size="1.778" layer="96" font="vector" rot="R90" align="top-center"/>
 </instance>
-<instance part="G1" gate="G$1" x="-152.4" y="134.62" rot="R90">
-<attribute name="NAME" x="-155.575" y="128.905" size="1.778" layer="95" rot="R90"/>
-<attribute name="VALUE" x="-147.32" y="128.905" size="1.778" layer="96" rot="R90"/>
+<instance part="G1" gate="G$1" x="-213.36" y="134.62" rot="R90">
+<attribute name="NAME" x="-216.535" y="128.905" size="1.778" layer="95" rot="R90"/>
+<attribute name="VALUE" x="-208.28" y="128.905" size="1.778" layer="96" rot="R90"/>
 </instance>
-<instance part="IC1" gate="A1" x="-116.84" y="142.24">
-<attribute name="NAME" x="-124.46" y="147.955" size="1.778" layer="95"/>
-<attribute name="VALUE" x="-124.46" y="145.415" size="1.778" layer="96"/>
+<instance part="IC1" gate="A1" x="-177.8" y="142.24">
+<attribute name="NAME" x="-185.42" y="147.955" size="1.778" layer="95"/>
+<attribute name="VALUE" x="-185.42" y="145.415" size="1.778" layer="96"/>
 </instance>
 <instance part="R2" gate="G$1" x="-30.48" y="63.5" rot="R90">
@@
 <attribute name="VALUE" x="-86.36" y="116.84" size="1.778" layer="96"/>
 </instance>
+<instance part="Y1" gate="G$1" x="-142.24" y="99.06">
+<attribute name="NAME" x="-142.24" y="101.092" size="1.778" layer="95" font="vector" align="bottom-center"/>
+<attribute name="VALUE" x="-142.24" y="97.028" size="1.778" layer="96" font="vector" align="top-center"/>
+</instance>
+<instance part="C1" gate="G$1" x="-144.78" y="86.36">
+<attribute name="NAME" x="-143.256" y="89.281" size="1.778" layer="95" font="vector"/>
+<attribute name="VALUE" x="-143.256" y="84.201" size="1.778" layer="96" font="vector"/>
+</instance>
+<instance part="C2" gate="G$1" x="-134.62" y="86.36">
+<attribute name="NAME" x="-133.096" y="89.281" size="1.778" layer="95" font="vector"/>
+<attribute name="VALUE" x="-133.096" y="84.201" size="1.778" layer="96" font="vector"/>
+</instance>
 </instances>
 <busses>
@@
 <segment>
 <pinref part="G1" gate="G$1" pin="+"/>
-<wire x1="-152.4" y1="147.32" x2="-152.4" y2="152.4" width="0.1524" layer="91"/>
+<wire x1="-213.36" y1="147.32" x2="-213.36" y2="152.4" width="0.1524" layer="91"/>
 <pinref part="IC1" gate="A1" pin="VI"/>
-<wire x1="-152.4" y1="152.4" x2="-127" y2="152.4" width="0.1524" layer="91"/>
-<wire x1="-127" y1="152.4" x2="-127" y2="142.24" width="0.1524" layer="91"/>
-<junction x="-127" y="142.24"/>
-<label x="-127" y="142.24" size="1.778" layer="95" rot="R180" xref="yes"/>
+<wire x1="-213.36" y1="152.4" x2="-187.96" y2="152.4" width="0.1524" layer="91"/>
+<wire x1="-187.96" y1="152.4" x2="-187.96" y2="142.24" width="0.1524" layer="91"/>
+<junction x="-187.96" y="142.24"/>
+<label x="-187.96" y="142.24" size="1.778" layer="95" rot="R180" xref="yes"/>
 </segment>
 </net>
@@
 <segment>
 <pinref part="IC1" gate="A1" pin="VO"/>
-<junction x="-106.68" y="142.24"/>
-<label x="-106.68" y="142.24" size="1.778" layer="95" xref="yes"/>
+<junction x="-167.64" y="142.24"/>
+<label x="-167.64" y="142.24" size="1.778" layer="95" xref="yes"/>
 </segment>
 <segment>
@@
 <segment>
 <pinref part="G1" gate="G$1" pin="-"/>
-<wire x1="-152.4" y1="121.92" x2="-152.4" y2="116.84" width="0.1524" layer="91"/>
-<wire x1="-152.4" y1="116.84" x2="-116.84" y2="116.84" width="0.1524" layer="91"/>
+<wire x1="-213.36" y1="121.92" x2="-213.36" y2="116.84" width="0.1524" layer="91"/>
+<wire x1="-213.36" y1="116.84" x2="-177.8" y2="116.84" width="0.1524" layer="91"/>
 <pinref part="IC1" gate="A1" pin="GND"/>
-<wire x1="-116.84" y1="116.84" x2="-116.84" y2="134.62" width="0.1524" layer="91"/>
-<junction x="-116.84" y="116.84"/>
-<junction x="-116.84" y="116.84"/>
-<label x="-116.84" y="116.84" size="1.778" layer="95" rot="R270" xref="yes"/>
+<wire x1="-177.8" y1="116.84" x2="-177.8" y2="134.62" width="0.1524" layer="91"/>
+<junction x="-177.8" y="116.84"/>
+<junction x="-177.8" y="116.84"/>
+<label x="-177.8" y="116.84" size="1.778" layer="95" rot="R270" xref="yes"/>
 <pinref part="IC2" gate="G$1" pin="GND"/>
-<wire x1="-116.84" y1="116.84" x2="-116.84" y2="81.28" width="0.1524" layer="91"/>
-<wire x1="-116.84" y1="81.28" x2="-104.14" y2="81.28" width="0.1524" layer="91"/>
-<junction x="-116.84" y="134.62"/>
-<label x="-116.84" y="134.62" size="1.778" layer="95" xref="yes"/>
+<wire x1="-177.8" y1="116.84" x2="-177.8" y2="81.28" width="0.1524" layer="91"/>
+<wire x1="-177.8" y1="81.28" x2="-104.14" y2="81.28" width="0.1524" layer="91"/>
+<junction x="-177.8" y="134.62"/>
+<label x="-177.8" y="134.62" size="1.778" layer="95" xref="yes"/>
 <junction x="-104.14" y="81.28"/>
 <label x="-104.14" y="81.28" size="1.778" layer="95" rot="R90" xref="yes"/>
@@
 <junction x="-104.14" y="106.68"/>
 <label x="-104.14" y="106.68" size="1.778" layer="95" rot="R180" xref="yes"/>
+</segment>
+<segment>
+<pinref part="C1" gate="G$1" pin="2"/>
+<junction x="-144.78" y="83.82"/>
+<label x="-144.78" y="83.82" size="1.778" layer="95" rot="R180" xref="yes"/>
+</segment>
+<segment>
+<pinref part="C2" gate="G$1" pin="2"/>
+<junction x="-134.62" y="83.82"/>
+<label x="-134.62" y="83.82" size="1.778" layer="95" xref="yes"/>
 </segment>
 </net>
@@
 </segment>
 </net>
+<net name="N$1" class="0">
+<segment>
+<pinref part="Y1" gate="G$1" pin="1"/>
+<wire x1="-144.78" y1="111.76" x2="-144.78" y2="99.06" width="0.1524" layer="91"/>
+<pinref part="IC2" gate="G$1" pin="PB6(XTAL1/TOSC1/PCI6)"/>
+<wire x1="-104.14" y1="93.98" x2="-114.3" y2="93.98" width="0.1524" layer="91"/>
+<wire x1="-114.3" y1="93.98" x2="-114.3" y2="111.76" width="0.1524" layer="91"/>
+<wire x1="-114.3" y1="111.76" x2="-144.78" y2="111.76" width="0.1524" layer="91"/>
+<wire x1="-144.78" y1="99.06" x2="-144.78" y2="91.44" width="0.1524" layer="91"/>
+<junction x="-144.78" y="99.06"/>
+<pinref part="C1" gate="G$1" pin="1"/>
+</segment>
+</net>
+<net name="N$2" class="0">
+<segment>
+<pinref part="Y1" gate="G$1" pin="2"/>
+<wire x1="-139.7" y1="99.06" x2="-134.62" y2="99.06" width="0.1524" layer="91"/>
+<wire x1="-134.62" y1="99.06" x2="-134.62" y2="91.44" width="0.1524" layer="91"/>
+<pinref part="C2" gate="G$1" pin="1"/>
+<pinref part="IC2" gate="G$1" pin="PB7(XTAL2/TOSC2/PCI7)"/>
+<wire x1="-104.14" y1="88.9" x2="-116.84" y2="88.9" width="0.1524" layer="91"/>
+<wire x1="-116.84" y1="88.9" x2="-116.84" y2="101.6" width="0.1524" layer="91"/>
+<wire x1="-116.84" y1="101.6" x2="-139.7" y2="101.6" width="0.1524" layer="91"/>
+<wire x1="-139.7" y1="101.6" x2="-139.7" y2="99.06" width="0.1524" layer="91"/>
+<junction x="-139.7" y="99.06"/>
+</segment>
+</net>

Commit message: Add files via upload
Parts:
- removed G1: AB9V, battery:AB9V
- added JP1: (no value), pinhead:PINHD-1X2
Connections:
- net 9V: now also JP1.1; no longer G1.+
- net GND: now also JP1.2; no longer G1.-
Changed lines of the file:
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@@
 <parts>
 <part name="R1" library="SparkFun-Resistors" library_urn="urn:adsk.eagle:library:532" deviceset="100KOHM" device="-0402-1/16W-1%" package3d_urn="urn:adsk.eagle:package:39657/1" value="4.7k"/>
-<part name="G1" library="battery" library_urn="urn:adsk.eagle:library:109" deviceset="AB9V" device="" package3d_urn="urn:adsk.eagle:package:4600/1"/>
 <part name="IC1" library="linear" library_urn="urn:adsk.eagle:library:262" deviceset="78*" device="T" package3d_urn="urn:adsk.eagle:package:16414/1" technology="05"/>
 <part name="R2" library="SparkFun-Resistors" library_urn="urn:adsk.eagle:library:532" deviceset="100KOHM" device="-0402-1/16W-1%" package3d_urn="urn:adsk.eagle:package:39657/1" value="150"/>
@@
 <part name="C1" library="SparkFun-Capacitors" library_urn="urn:adsk.eagle:library:510" deviceset="22PF" device="-0603-50V-5%" package3d_urn="urn:adsk.eagle:package:37414/1" value="22pF"/>
 <part name="C2" library="SparkFun-Capacitors" library_urn="urn:adsk.eagle:library:510" deviceset="22PF" device="-0603-50V-5%" package3d_urn="urn:adsk.eagle:package:37414/1" value="22pF"/>
+<part name="JP1" library="pinhead" library_urn="urn:adsk.eagle:library:325" deviceset="PINHD-1X2" device="" package3d_urn="urn:adsk.eagle:package:22435/2"/>
 </parts>
 <sheets>
@@
 <attribute name="NAME" x="-85.344" y="134.62" size="1.778" layer="95" font="vector" rot="R90" align="bottom-center"/>
 <attribute name="VALUE" x="-82.296" y="134.62" size="1.778" layer="96" font="vector" rot="R90" align="top-center"/>
-</instance>
-<instance part="G1" gate="G$1" x="-213.36" y="134.62" rot="R90">
-<attribute name="NAME" x="-216.535" y="128.905" size="1.778" layer="95" rot="R90"/>
-<attribute name="VALUE" x="-208.28" y="128.905" size="1.778" layer="96" rot="R90"/>
 </instance>
 <instance part="IC1" gate="A1" x="-177.8" y="142.24">
@@
 <attribute name="VALUE" x="-133.096" y="84.201" size="1.778" layer="96" font="vector"/>
 </instance>
+<instance part="JP1" gate="G$1" x="-213.36" y="134.62">
+<attribute name="NAME" x="-219.71" y="140.335" size="1.778" layer="95"/>
+<attribute name="VALUE" x="-219.71" y="129.54" size="1.778" layer="96"/>
+</instance>
 </instances>
 <busses>
@@
 <net name="9V" class="0">
 <segment>
-<pinref part="G1" gate="G$1" pin="+"/>
-<wire x1="-213.36" y1="147.32" x2="-213.36" y2="152.4" width="0.1524" layer="91"/>
 <pinref part="IC1" gate="A1" pin="VI"/>
 <wire x1="-213.36" y1="152.4" x2="-187.96" y2="152.4" width="0.1524" layer="91"/>
@@
 <junction x="-187.96" y="142.24"/>
 <label x="-187.96" y="142.24" size="1.778" layer="95" rot="R180" xref="yes"/>
+<pinref part="JP1" gate="G$1" pin="1"/>
+<wire x1="-215.9" y1="137.16" x2="-213.36" y2="137.16" width="0.1524" layer="91"/>
+<wire x1="-213.36" y1="137.16" x2="-213.36" y2="152.4" width="0.1524" layer="91"/>
 </segment>
 </net>
@@
 <net name="GND" class="0">
 <segment>
-<pinref part="G1" gate="G$1" pin="-"/>
-<wire x1="-213.36" y1="121.92" x2="-213.36" y2="116.84" width="0.1524" layer="91"/>
 <wire x1="-213.36" y1="116.84" x2="-177.8" y2="116.84" width="0.1524" layer="91"/>
 <pinref part="IC1" gate="A1" pin="GND"/>
@@
 <junction x="-104.14" y="81.28"/>
 <label x="-104.14" y="81.28" size="1.778" layer="95" rot="R90" xref="yes"/>
+<pinref part="JP1" gate="G$1" pin="2"/>
+<wire x1="-215.9" y1="134.62" x2="-213.36" y2="134.62" width="0.1524" layer="91"/>
+<wire x1="-213.36" y1="134.62" x2="-213.36" y2="116.84" width="0.1524" layer="91"/>
 </segment>
 <segment>
